Commit message: fixed ros2 incompatible frame names

File: duckiebot_interface/urdf/duckiebot.urdf (robot description, URDF)
Before this commit: robot duckiebot, 17 links, 16 joints
Links:
- removed link /duckiebot/back_bumper
- removed link /duckiebot/base
- removed link /duckiebot/bottom_plate
- removed link /duckiebot/camera_frame
- removed link /duckiebot/camera_mount
- removed link /duckiebot/camera_optical_frame
- removed link /duckiebot/camera_support
- removed link /duckiebot/caster_wheel
- removed link /duckiebot/footprint
- removed link /duckiebot/front_bumper
- removed link /duckiebot/left_motor
- removed link /duckiebot/left_wheel
- removed link /duckiebot/left_wheel_axis
- removed link /duckiebot/right_motor
- removed link /duckiebot/right_wheel
- removed link /duckiebot/right_wheel_axis
- removed link /duckiebot/top_plate
- added link duckiebot/back_bumper; visual mesh filename=package://duckietown/urdf/meshes/duckiebot/DB18/back_bumper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
- added link duckiebot/base
- added link duckiebot/bottom_plate; visual mesh filename=package://duckietown/urdf/meshes/duckiebot/DB18/bottom_plat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
- added link duckiebot/camera_frame; visual mesh filename=package://duckietown/urdf/meshes/duckiebot/DB18/fish_eye_ca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
- added link duckiebot/camera_mount; visual mesh filename=package://duckietown/urdf/meshes/duckiebot/DB18/camera_moun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
- added link duckiebot/camera_optical_frame
- added link duckiebot/camera_support
- added link duckiebot/caster_wheel; visual mesh filename=package://duckietown/urdf/meshes/duckiebot/DB18/caster_whee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
- added link duckiebot/footprint
- added link duckiebot/front_bumper; visual mesh filename=package://duckietown/urdf/meshes/duckiebot/DB18/front_bumpe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
- added link duckiebot/left_motor; visual mesh filename=package://duckietown/urdf/meshes/duckiebot/DB18/motor.dae
- added link duckiebot/left_wheel; visual mesh filename=package://duckietown/urdf/meshes/duckiebot/DB18/wheel.dae
- added link duckiebot/left_wheel_axis
- added link duckiebot/right_motor; visual mesh filename=package://duckietown/urdf/meshes/duckiebot/DB18/motor.dae
- added link duckiebot/right_wheel; visual mesh filename=package://duckietown/urdf/meshes/duckiebot/DB18/wheel.dae
- added link duckiebot/right_wheel_axis
- added link duckiebot/top_plate; visual mesh filename=package://duckietown/urdf/meshes/duckiebot/DB18/top_plate.d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
Joints:
- joint duckiebot_base_to_bottom_plate: child /duckiebot/bottom_plate -> duckiebot/bottom_plate; parent /duckiebot/base -> duckiebot/base
- joint duckiebot_base_to_left_motor: child /duckiebot/left_motor -> duckiebot/left_motor; parent /duckiebot/base -> duckiebot/base
- joint duckiebot_base_to_right_motor: child /duckiebot/right_motor -> duckiebot/right_motor; parent /duckiebot/base -> duckiebot/base
- joint duckiebot_bottom_plate_to_back_bumper: child /duckiebot/back_bumper -> duckiebot/back_bumper; parent /duckiebot/bottom_plate -> duckiebot/bottom_plate
- joint duckiebot_bottom_plate_to_caster_wheel: child /duckiebot/caster_wheel -> duckiebot/caster_wheel; parent /duckiebot/bottom_plate -> duckiebot/bottom_plate
- joint duckiebot_bottom_plate_to_front_bumper: child /duckiebot/front_bumper -> duckiebot/front_bumper; parent /duckiebot/bottom_plate -> duckiebot/bottom_plate
- joint duckiebot_bottom_plate_to_top_plate: child /duckiebot/top_plate -> duckiebot/top_plate; parent /duckiebot/bottom_plate -> duckiebot/bottom_plate
- joint duckiebot_camera_frame_to_camera_optical_frame: child /duckiebot/camera_optical_frame -> duckiebot/camera_optical_frame; parent /duckiebot/camera_frame -> duckiebot/camera_frame
- joint duckiebot_camera_mount_to_camera_support: child /duckiebot/camera_support -> duckiebot/camera_support; parent /duckiebot/camera_mount -> duckiebot/camera_mount
- joint duckiebot_camera_support_to_camera_frame: child /duckiebot/camera_frame -> duckiebot/camera_frame; parent /duckiebot/camera_support -> duckiebot/camera_support
- joint duckiebot_footprint_to_base: child /duckiebot/base -> duckiebot/base; parent /duckiebot/footprint -> duckiebot/footprint
- joint duckiebot_left_motor_to_left_wheel: child /duckiebot/left_wheel_axis -> duckiebot/left_wheel_axis; parent /duckiebot/left_motor -> duckiebot/left_motor
- joint duckiebot_left_wheel_axis_to_left_wheel: child /duckiebot/left_wheel -> duckiebot/left_wheel; parent /duckiebot/left_wheel_axis -> duckiebot/left_wheel_axis
- joint duckiebot_right_motor_to_right_wheel: child /duckiebot/right_wheel_axis -> duckiebot/right_wheel_axis; parent /duckiebot/right_motor -> duckiebot/right_motor
- joint duckiebot_right_wheel_axis_to_right_wheel: child /duckiebot/right_wheel -> duckiebot/right_wheel; parent /duckiebot/right_wheel_axis -> duckiebot/right_wheel_axis
- joint duckiebot_top_plate_to_camera_mount: child /duckiebot/camera_mount -> duckiebot/camera_mount; parent /duckiebot/top_plate -> duckiebot/top_plate
